File: bmi088-i2c-breakout.kicad_sch (KiCad schematic)
At the start: 0 parts

Commit message: modified:   bmi088-i2c-breakout.kicad_pcb
Parts:
- added C1, C2: 0.1μF, Capacitor_SMD:C_0201_0603Metric, symbol Device:C
- added J1, J2: Conn_01x04_Socket, Connector_PinHeader_2.54mm:PinHeader_1x04_P2.54mm_Vertical, symbol Connector:Conn_01x04_Socket
- added JP1, JP2: Jumper_2_Open, Capacitor_SMD:C_0201_0603Metric, symbol Jumper:Jumper_2_Open
- added R1, R2: 1.5kΩ, Capacitor_SMD:C_0201_0603Metric, symbol Device:R
- added U1: BMI088, Package_LGA:Bosch_LGA-16_4.5x3mm_P0.5mm_LayoutBorder7x1y_ClockwisePinNumbering, symbol Sensor_Motion:BMI088
Connections:
- new net: JP2.2 (B), R1.1
- new net: JP1.2 (B), R2.1
- new net 3V3: C1.1, C2.1, J2.1 (Pin_1), JP1.1 (A), JP2.1 (A), U1.3 (VDD), U1.7 (PS)
- new net GND: C1.2, C2.2, J2.2 (Pin_2), U1.10 (SDO2), U1.15 (SDO1), U1.2 (GNDA), U1.4 (GNDA), U1.6 (GNDIO)
- new net INT1: J1.1 (Pin_1), U1.16 (INT1)
- new net INT2: J1.2 (Pin_2), U1.1 (INT2)
- new net INT3: J1.3 (Pin_3), U1.12 (INT3)
- new net INT4: J1.4 (Pin_4), U1.13 (INT4)
- new net SCL: J2.3 (Pin_3), R1.2, U1.8 (SCK/SCL)
- new net SDA: J2.4 (Pin_4), R2.2, U1.9 (SDI/SDA)
- new net VDDIO: U1.11 (VDDIO)

Commit message: modified:   bmi088-i2c-breakout.kicad_pcb
Connections:
- net VDDIO is gone; now on net 3V3: U1.11 (VDDIO)
- net 3V3: now also J1.1 (Pin_1); no longer J2.1 (Pin_1)
- net INT1: now also J2.1 (Pin_1); no longer J1.1 (Pin_1)
- net INT2: now also J2.3 (Pin_3); no longer J1.2 (Pin_2)
- net INT3: now also J1.4 (Pin_4); no longer J1.3 (Pin_3)
- net INT4: now also J2.4 (Pin_4); no longer J1.4 (Pin_4)
- net SCL: now also J1.2 (Pin_2); no longer J2.3 (Pin_3)
- net SDA: now also J1.3 (Pin_3); no longer J2.4 (Pin_4)
Other:
- moved on the sheet: C1, C2
Changed lines of the file:
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@@
 	(paper "A4")
 	(junction
-		(at 80.01 124.46)
+		(at 186.69 100.33)
 		(diameter 0)
 		(color 0 0 0 0)
 	)
 	(junction
-		(at 93.98 124.46)
+		(at 172.72 97.79)
 		(diameter 0)
 		(color 0 0 0 0)
@@
 	(wire
 		(pts
-			(xy 137.16 97.79) (xy 142.24 97.79)
+			(xy 137.16 97.79) (xy 172.72 97.79)
 		)
 		(stroke
@@
 	(wire
 		(pts
-			(xy 80.01 124.46) (xy 80.01 128.27)
-		)
-		(stroke
-			(width 0)
-			(type default)
-		)
-	)
-	(wire
-		(pts
-			(xy 80.01 147.32) (xy 85.09 147.32)
+			(xy 172.72 92.71) (xy 172.72 97.79)
+		)
+		(stroke
+			(width 0)
+			(type default)
+		)
+	)
+	(wire
+		(pts
+			(xy 172.72 123.19) (xy 177.8 123.19)
 		)
 		(stroke
@@
 	(wire
 		(pts
-			(xy 74.93 124.46) (xy 80.01 124.46)
-		)
-		(stroke
-			(width 0)
-			(type default)
-		)
-	)
-	(wire
-		(pts
 			(xy 152.4 127) (xy 160.02 127)
 		)
@@
 	(wire
 		(pts
-			(xy 80.01 135.89) (xy 80.01 147.32)
-		)
-		(stroke
-			(width 0)
-			(type default)
-		)
-	)
-	(wire
-		(pts
-			(xy 93.98 135.89) (xy 93.98 147.32)
+			(xy 172.72 111.76) (xy 172.72 123.19)
+		)
+		(stroke
+			(width 0)
+			(type default)
+		)
+	)
+	(wire
+		(pts
+			(xy 186.69 111.76) (xy 186.69 123.19)
 		)
 		(stroke
@@
 	(wire
 		(pts
-			(xy 93.98 147.32) (xy 99.06 147.32)
+			(xy 186.69 123.19) (xy 191.77 123.19)
 		)
 		(stroke
@@
 	(wire
 		(pts
-			(xy 142.24 100.33) (xy 147.32 100.33)
-		)
-		(stroke
-			(width 0)
-			(type default)
-		)
-	)
-	(wire
-		(pts
-			(xy 88.9 124.46) (xy 93.98 124.46)
-		)
-		(stroke
-			(width 0)
-			(type default)
-		)
-	)
-	(wire
-		(pts
-			(xy 93.98 116.84) (xy 99.06 116.84)
-		)
-		(stroke
-			(width 0)
-			(type default)
-		)
-	)
-	(wire
-		(pts
-			(xy 93.98 116.84) (xy 93.98 124.46)
+			(xy 142.24 100.33) (xy 186.69 100.33)
+		)
+		(stroke
+			(width 0)
+			(type default)
+		)
+	)
+	(wire
+		(pts
+			(xy 186.69 92.71) (xy 191.77 92.71)
+		)
+		(stroke
+			(width 0)
+			(type default)
+		)
+	)
+	(wire
+		(pts
+			(xy 186.69 92.71) (xy 186.69 100.33)
 		)
 		(stroke
@@
 	(wire
 		(pts
-			(xy 80.01 116.84) (xy 85.09 116.84)
+			(xy 172.72 92.71) (xy 177.8 92.71)
 		)
 		(stroke
@@
 	(wire
 		(pts
+			(xy 186.69 100.33) (xy 186.69 104.14)
+		)
+		(stroke
+			(width 0)
+			(type default)
+		)
+	)
+	(wire
+		(pts
 			(xy 92.71 81.28) (xy 92.71 82.55)
 		)
@@
 	(wire
 		(pts
-			(xy 80.01 116.84) (xy 80.01 124.46)
-		)
-		(stroke
-			(width 0)
-			(type default)
-		)
-	)
-	(wire
-		(pts
 			(xy 92.71 99.06) (xy 97.79 99.06)
 		)
@@
 	(wire
 		(pts
+			(xy 172.72 97.79) (xy 172.72 104.14)
+		)
+		(stroke
+			(width 0)
+			(type default)
+		)
+	)
+	(wire
+		(pts
 			(xy 121.92 116.84) (xy 127 116.84)
-		)
-		(stroke
-			(width 0)
-			(type default)
-		)
-	)
-	(wire
-		(pts
-			(xy 93.98 124.46) (xy 93.98 128.27)
 		)
 		(stroke
@@
 		)
 	)
-	(label "SCL"
-		(at 157.48 147.32 0)
-		(effects
-			(font
-				(size 1.27 1.27)
-			)
-			(justify left bottom)
-		)
-	)
 	(label "INT3"
 		(at 153.67 121.92 0)
@@
 		)
 	)
-	(label "INT4"
+	(label "INT3"
 		(at 158.75 163.83 0)
 		(effects
@@
 		)
 	)
+	(label "INT4"
+		(at 157.48 149.86 0)
+		(effects
+			(font
+				(size 1.27 1.27)
+			)
+			(justify left bottom)
+		)
+	)
 	(label "GND"
-		(at 81.28 147.32 0)
+		(at 173.99 123.19 0)
 		(effects
 			(font
@@
 		)
 	)
-	(label "VDDIO"
-		(at 143.51 100.33 0)
-		(effects
-			(font
-				(size 1.27 1.27)
-			)
-			(justify left bottom)
-		)
-	)
 	(label "GND"
 		(at 121.92 121.92 0)
@@
 		)
 	)
+	(label "SCL"
+		(at 158.75 158.75 0)
+		(effects
+			(font
+				(size 1.27 1.27)
+			)
+			(justify left bottom)
+		)
+	)
 	(label "SDA"
 		(at 121.92 119.38 0)
@@
 		)
 	)
-	(label "SDA"
-		(at 157.48 149.86 0)
-		(effects
-			(font
-				(size 1.27 1.27)
-			)
-			(justify left bottom)
-		)
-	)
 	(label "3V3"
-		(at 95.25 116.84 0)
-		(effects
-			(font
-				(size 1.27 1.27)
-			)
-			(justify left bottom)
-		)
-	)
-	(label "INT2"
-		(at 158.75 158.75 0)
+		(at 187.96 92.71 0)
 		(effects
 			(font
@@
 	)
 	(label "3V3"
-		(at 80.01 116.84 0)
-		(effects
-			(font
-				(size 1.27 1.27)
-			)
-			(justify left bottom)
-		)
-	)
-	(label "INT1"
+		(at 172.72 92.71 0)
+		(effects
+			(font
+				(size 1.27 1.27)
+			)
+			(justify left bottom)
+		)
+	)
+	(label "3V3"
 		(at 158.75 156.21 0)
 		(effects
@@
 		)
 	)
-	(label "3V3"
+	(label "INT1"
 		(at 157.48 142.24 0)
 		(effects
@@
 		)
 	)
-	(label "VDD"
-		(at 137.16 97.79 0)
-		(effects
-			(font
-				(size 1.27 1.27)
-			)
-			(justify left bottom)
-		)
-	)
-	(label "INT3"
+	(label "SDA"
 		(at 158.75 161.29 0)
 		(effects
@@
 		)
 	)
-	(label "VDD"
-		(at 74.93 124.46 0)
-		(effects
-			(font
-				(size 1.27 1.27)
-			)
-			(justify left bottom)
-		)
-	)
-	(label "VDDIO"
-		(at 87.63 124.46 0)
+	(label "INT2"
+		(at 157.48 147.32 0)
 		(effects
 			(font
@@
 	)
 	(label "GND"
-		(at 95.25 147.32 0)
+		(at 187.96 123.19 0)
 		(effects
 			(font
@@
 	(symbol
 		(lib_id "Device:C")
-		(at 93.98 132.08 0)
+		(at 186.69 107.95 0)
 		(unit 1)
 		(body_style 1)
@@
 		(fields_autoplaced yes)
 		(property "Reference" "C2"
-			(at 97.79 130.8099 0)
+			(at 190.5 106.6799 0)
 			(show_name no)
 			(do_not_autoplace no)
@@
 		)
 		(property "Value" "0.1μF"
-			(at 97.79 133.3499 0)
+			(at 190.5 109.2199 0)
 			(show_name no)
 			(do_not_autoplace no)
@@
 		)
 		(property "Footprint" "Capacitor_SMD:C_0201_0603Metric"
-			(at 94.9452 135.89 0)
+			(at 187.6552 111.76 0)
 			(hide yes)
 			(show_name no)
@@
 		)
 		(property "Datasheet" ""
-			(at 93.98 132.08 0)
+			(at 186.69 107.95 0)
 			(hide yes)
 			(show_name no)
@@
 		)
 		(property "Description" "Unpolarized capacitor"
-			(at 93.98 132.08 0)
+			(at 186.69 107.95 0)
 			(hide yes)
 			(show_name no)
@@
 	(symbol
 		(lib_id "Device:C")
-		(at 80.01 132.08 0)
+		(at 172.72 107.95 0)
 		(unit 1)
 		(body_style 1)
@@
 		(fields_autoplaced yes)
 		(property "Reference" "C1"
-			(at 83.82 130.8099 0)
+			(at 176.53 106.6799 0)
 			(show_name no)
 			(do_not_autoplace no)
@@
 		)
 		(property "Value" "0.1μF"
-			(at 83.82 133.3499 0)
+			(at 176.53 109.2199 0)
 			(show_name no)
 			(do_not_autoplace no)
@@
 		)
 		(property "Footprint" "Capacitor_SMD:C_0201_0603Metric"
-			(at 80.9752 135.89 0)
+			(at 173.6852 111.76 0)
 			(hide yes)
 			(show_name no)
@@
 		)
 		(property "Datasheet" ""
-			(at 80.01 132.08 0)
+			(at 172.72 107.95 0)
 			(hide yes)
 			(show_name no)
@@
 		)
 		(property "Description" "Unpolarized capacitor"
-			(at 80.01 132.08 0)
-			(hide yes)
-			(show_name no)
+			(at 172.72 107.95 0)
+			(hide yes)
+			(show_name no)

Commit message: Fixed mis-labeled resistors
Parts:
- JP1: renamed from JP2; value Jumper_2_Open -> Jumper_1_Open; footprint Capacitor_SMD:C_0201_0603Metric -> Resistor_SMD:C_0201_0603Metric
- JP2: renamed from JP1; footprint Capacitor_SMD:C_0201_0603Metric -> Resistor_SMD:C_0201_0603Metric
- R1, R2: footprint Capacitor_SMD:C_0201_0603Metric -> Resistor_SMD:R_0201_0603Metric
Changed lines of the file:
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@@
 			)
 		)
-		(property "Footprint" "Capacitor_SMD:C_0201_0603Metric"
+		(property "Footprint" "Resistor_SMD:R_0201_0603Metric"
 			(at 80.772 86.36 90)
 			(hide yes)
@@
 		(dnp no)
 		(fields_autoplaced yes)
-		(property "Reference" "JP1"
+		(property "Reference" "JP2"
 			(at 95.25 74.9299 90)
 			(hide yes)
@@
 			)
 		)
-		(property "Footprint" "Capacitor_SMD:C_0201_0603Metric"
+		(property "Footprint" "Resistor_SMD:C_0201_0603Metric"
 			(at 92.71 76.2 0)
 			(hide yes)
@@
 			(project "bmi088-i2c-breakout"
 				(path "/62fce77e-fdaf-4ea6-889e-53ca4188e9b9"
-					(reference "JP1")
+					(reference "JP2")
 					(unit 1)
 				)
@@
 		(dnp no)
 		(fields_autoplaced yes)
-		(property "Reference" "JP2"
+		(property "Reference" "JP1"
 			(at 85.09 74.9299 90)
 			(hide yes)
@@
 			)
 		)
-		(property "Value" "Jumper_2_Open"
+		(property "Value" "Jumper_1_Open"
 			(at 85.09 77.4699 90)
 			(hide yes)
@@
 			)
 		)
-		(property "Footprint" "Capacitor_SMD:C_0201_0603Metric"
+		(property "Footprint" "Resistor_SMD:C_0201_0603Metric"
 			(at 82.55 76.2 0)
 			(hide yes)
@@
 			(project "bmi088-i2c-breakout"
 				(path "/62fce77e-fdaf-4ea6-889e-53ca4188e9b9"
-					(reference "JP2")
+					(reference "JP1")
 					(unit 1)
 				)
@@
 			)
 		)
-		(property "Footprint" "Capacitor_SMD:C_0201_0603Metric"
+		(property "Footprint" "Resistor_SMD:R_0201_0603Metric"
 			(at 90.932 86.36 90)
 			(hide yes)
