File: bmi088-i2c-breakout.kicad_pcb (KiCad board)
At the start: 2 copper layers, 14.2 x 10.1 mm, 11 parts, among them J1 Conn_01x04_Socket, J2 Conn_01x04_Socket, U1 BMI088

Commit message: modified:   bmi088-i2c-breakout.kicad_pcb
Parts:
- removed the G*** at (147.9, 95.5)
- removed the G*** at (152.5, 94.3)
- added G***: LOGO, LOGO, F.Cu at (148.1, 95.8)
- added G***: LOGO, LOGO, B.Cu at (151.4, 94.2)

Commit message: modified:   bmi088-i2c-breakout.kicad_pcb
Parts:
- removed the G*** at (148.1, 95.8)
- moved G*** 0.10 mm to (151.5, 94.3)
Other:
- board text added: "BobbieBots IMU-BMI088-V1.0"
- board text added: "IMU-BMI088-V1.0"
