File: thru-hole/bmi088-i2c-breakout.kicad_pcb (KiCad board)
At the start: 2 copper layers, 14.2 x 10.1 mm, 10 parts, among them J1 Conn_01x04_Socket, J2 Conn_01x04_Socket, U1 BMI088

Commit message: modified:   thru-hole/bmi088-i2c-breakout.kicad_pcb
Other:
- board size 14.2 x 10.1 mm -> 16.5 x 10.1 mm
Changed lines of the file:
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@@
 	)
 	(gr_rect
-		(start 144.85 89.4)
-		(end 159 99.5)
+		(start 143.73 89.4)
+		(end 160.23 99.5)
 		(stroke
 			(width 0.05)
